File: Hardware/Motherboard/Motherboard.kicad_sch (KiCad schematic)
At the start: 0 parts

Commit message: Day 6
Parts:
- added U1: STM32F072C8Tx, Package_QFP:LQFP-48_7x7mm_P0.5mm, symbol MCU_ST_STM32F0:STM32F072C8Tx
Connections:
- new net: U1.23 (VSS), U1.35 (VSS), U1.47 (VSS)
Changed lines of the file:
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@@
 	(generator_version "9.0")
 	(paper "A4")
+	(symbol
+		(lib_id "MCU_ST_STM32F0:STM32F072C8Tx")
+		(at 95.25 100.33 0)
+		(unit 1)
+		(exclude_from_sim no)
+		(in_bom yes)
+		(on_board yes)
+		(dnp no)
+		(fields_autoplaced yes)
+		(property "Reference" "U1"
+			(at 99.9333 140.97 0)
+			(effects
+				(font
+					(size 1.27 1.27)
+				)
+				(justify left)
+			)
+		)
+		(property "Value" "STM32F072C8Tx"
+			(at 99.9333 143.51 0)
+			(effects
+				(font
+					(size 1.27 1.27)
+				)
+				(justify left)
+			)
+		)
+		(property "Footprint" "Package_QFP:LQFP-48_7x7mm_P0.5mm"
+			(at 80.01 138.43 0)
+			(effects
+				(font
+					(size 1.27 1.27)
+				)
+				(justify right)
+				(hide yes)
+			)
+		)
+		(property "Datasheet" "https://www.st.com/resource/en/datasheet/stm32f072c8.pdf"
+			(at 95.25 100.33 0)
+			(effects
+				(font
+					(size 1.27 1.27)
+				)
+				(hide yes)
+			)
+		)
+		(property "Description" "STMicroelectronics Arm Cortex-M0 MCU, 64KB flash, 16KB RAM, 48 MHz, 2.0-3.6V, 37 GPIO, LQFP48"
+			(at 95.25 100.33 0)
+			(effects
+				(font
+					(size 1.27 1.27)
+				)
+				(hide yes)
+			)
+		)
+		(pin "7"
+		)
+		(pin "44"
+		)
+		(pin "5"
+		)
+		(pin "6"
+		)
+		(pin "2"
+		)
+		(pin "3"
+		)
+		(pin "4"
+		)
+		(pin "18"
+		)
+		(pin "19"
+		)
+		(pin "20"
+		)
+		(pin "39"
+		)
+		(pin "40"
+		)
+		(pin "41"
+		)
+		(pin "42"
+		)
+		(pin "43"
+		)
+		(pin "45"
+		)
+		(pin "46"
+		)
+		(pin "21"
+		)
+		(pin "22"
+		)
+		(pin "25"
+		)
+		(pin "26"
+		)
+		(pin "27"
+		)
+		(pin "28"
+		)
+		(pin "1"
+		)
+		(pin "24"
+		)
+		(pin "48"
+		)
+		(pin "23"
+		)
+		(pin "35"
+		)
+		(pin "47"
+		)
+		(pin "9"
+		)
+		(pin "8"
+		)
+		(pin "36"
+		)
+		(pin "10"
+		)
+		(pin "11"
+		)
+		(pin "12"
+		)
+		(pin "13"
+		)
+		(pin "14"
+		)
+		(pin "15"
+		)
+		(pin "16"
+		)
+		(pin "17"
+		)
+		(pin "29"
+		)
+		(pin "30"
+		)
+		(pin "31"
+		)
+		(pin "32"
+		)
+		(pin "33"
+		)
+		(pin "34"
+		)
+		(pin "37"
+		)
+		(pin "38"
+		)
+		(instances
+			(project ""
+				(path "/5996147d-8cbf-4196-8f5c-8df746bcf8cf"
+					(reference "U1")
+					(unit 1)
+				)
+			)
+		)
+	)
 	(sheet_instances
 		(path "/"
