File: Hardware/Motor_Driver/Motor_Driver.kicad_pcb (KiCad board)
At the start: 4 copper layers, 50.8 x 32.2 mm, 45 parts, among them J1 Conn_PWR, J2 Conn_MB, J3 Conn_SENSORS, J4 Conn_MOTOR, Q1 CSD87333Q3D, Q2 CSD87333Q3D, Q3 CSD87333Q3D, U1 DRV8320RS

Commit message: Day 6
Parts:
- J2: footprint Connector_PinHeader_2.54mm:PinHeader_2x06_P2.54mm_Vertical -> Connector_PinSocket_2.54mm:PinSocket_2x08_P2.54mm_Vertical
- moved R2 36.4 mm to (139.1, 104.2), turned to 180 degrees
- moved C1 34.6 mm to (139.1, 105.7), turned to 180 degrees
- moved C7 12.6 mm to (127.7, 102.0)
- moved J2 4.53 mm to (134.2, 97.4)
- moved R5 1.20 mm to (145.8, 102.5)
- moved R1 0.83 mm to (142.8, 102.5)
Connections:
- J2 pad 1: +5V -> VM
- J2 pad 10: /SDO -> /SDI
- J2 pad 11: /TEMP -> /SDO
- J2 pad 12: GND -> /TEMP
- J2 pad 2: /EN -> +5V
- J2 pad 3: /PWM -> /EN
- J2 pad 4: /DIR -> /PWM
- J2 pad 5: /BRAKE -> /DIR
- J2 pad 6: /FAULT -> /BRAKE
- J2 pad 7: /CS -> /FAULT
- J2 pad 8: /CLK -> /CS
- J2 pad 9: /SDI -> /CLK
Routing:
- net /HALL_C: track 69.7 -> 0.00 mm, vias 2 -> 0
- net +5V: track 58.0 -> 0.00 mm
- net /HALL_B: track 57.7 -> 0.00 mm, vias 2 -> 0
- net /HALL_A: track 51.2 -> 0.00 mm, vias 2 -> 0
- net /TEMP: track 35.6 -> 0.00 mm
- net /Phase_A.GL: track 25.6 -> 0.00 mm, vias 2 -> 1
- net /Phase_C.GL: track 23.0 -> 0.00 mm, vias 2 -> 1
- net /DIR: track 21.5 -> 0.00 mm
- net /Phase_B.GL: track 19.6 -> 0.00 mm, vias 2 -> 1
- net /Phase_A.SH: track 19.1 -> 0.00 mm, vias 2 -> 1
- net +3V3: track 19.0 -> 0.00 mm, vias 3 -> 0
- net Net-(D1-K): track 18.9 -> 0.00 mm
- net /Phase_C.SH: track 17.8 -> 0.00 mm, vias 2 -> 1
- net /Phase_B.SH: track 16.4 -> 0.00 mm, vias 2 -> 1
- net /Phase_B.GH: track 15.6 -> 0.00 mm, vias 2 -> 1
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